File: projects/Adapter Board/Adapter Board.sch (EAGLE design)
At the start: 38 parts

Commit message: Rev.2 Commit
Joined common pads, removed orphaned pads, aligned passive 0805s. More
room to solder QFN. Full rectangular board.
Parts:
- C1, C2, C3, C4, C6, C8, C9: value 220pF -> 10uF; device SparkFun-Passives:CAP0805 -> SparkFun-Capacitors:10UF-6.3V-20%(1206)
- C10: value 220pF -> 2.2uF; device SparkFun-Passives:CAP0805 -> SparkFun-Capacitors:CAP0805
- C11, C12: value 10uF -> 2.2uF; device SparkFun-Capacitors:10UF-6.3V-20%(1206) -> SparkFun-Capacitors:CAP0805
- C13: value 10uF -> 0.1uF; device SparkFun-Capacitors:10UF-6.3V-20%(1206) -> SparkFun-Capacitors:CAP0805
- C14, C15, C16: value 10uF -> 220pF; device SparkFun-Capacitors:10UF-6.3V-20%(1206) -> SparkFun-Passives:CAP0805
- C17: value 10uF -> 4.7uF; device SparkFun-Capacitors:10UF-6.3V-20%(1206) -> SparkFun-Capacitors:CAP0805
- C18: value 0.1uF -> 220pF; device SparkFun-Capacitors:CAP0805 -> SparkFun-Passives:CAP0805
- C20: value 4.7uF -> 220pF; device SparkFun-Capacitors:CAP0805 -> SparkFun-Passives:CAP0805
- C22, C23, C24: value 2.2uF -> 220pF; device SparkFun-Capacitors:CAP0805 -> SparkFun-Passives:CAP0805
- C25: value 100pF -> 220pF; device SparkFun-Capacitors:CAP0805 -> SparkFun-Passives:CAP0805
- C26: value 2700pF -> 220pF; device SparkFun-Capacitors:CAP0805 -> SparkFun-Passives:CAP0805
- C5: value 220pF -> 100pF; device SparkFun-Passives:CAP0805 -> SparkFun-Capacitors:CAP0805
- C7: value 220pF -> 2700pF; device SparkFun-Passives:CAP0805 -> SparkFun-Capacitors:CAP0805
- R1: value 1K -> 5.6K
- R2: value 5.6K -> 150K
- R3: value 66.5K -> 20K
- R4: value 150K -> 66.5K
- R5: value 20K -> 1K
- renumbered DIOD-S to D1, U$1 to F1, U$2 to F2, U$3 to U1, U$4 to I1
Connections:
- net BKLT-VCC: now also C1.1, C2.1, C3.1, C4.1, C6.1, C8.1, C9.1; no longer C11.1, C12.1, C14.1, C15.1, C16.1, C17.1, C18.1
- net BL-ANODE: now also C17.1, R2.2; no longer C20.1, R4.2
- net BL0: now also C26.1; no longer C1.1
- net BL1: now also C25.1; no longer C2.1
- net BL2: now also C24.1; no longer C3.1
- net BL3: now also C23.1; no longer C4.1
- net BL4: now also C22.1; no longer C5.1
- net BL5: now also C20.1; no longer C6.1
- net BL6: now also C18.1; no longer C7.1
- net BL7: now also C16.1; no longer C8.1
- net BL8: now also C15.1; no longer C9.1
- net BL9: now also C14.1; no longer C10.1
- net GND: now also C10.1, C11.1, C12.1, C22.2, C23.2, C24.2, R3.1, R4.2; no longer C10.2, C11.2, C12.2, C22.1, C23.1, C24.1, R3.2, R5.1
- net N$1: now also C5.1, R1.2; no longer C25.1, R2.2
- net N$10: now also C12.2, R5.1; no longer C24.2, R1.1
- net N$13: now also C7.1, R1.1; no longer C26.1, R2.1
- net N$16: now also R2.1, R3.2; no longer R4.1, R5.2
- net N$17: now also R4.1; no longer R3.1
- net N$4: now also C11.2; no longer C23.2
- net VDC1: now also C10.2, R5.2; no longer C22.2, R1.2
Other:
- moved on the sheet: C1, C10, C11, C12, C13, C14, C15, C16, C17, C18, C19, C2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
